Commit message: Aggiornato XACRO E Tabelle DH (Risolta Coincidenza Che jointRadius = boxSize/2)

File: urdf/manipolatoreRRP.urdf.xacro (robot description, xacro)
@@ -98,5 +98,5 @@
         <child link="RF1"/>
         <!-- DD Posizionamento In Cima Al Primo Link (Altezza L1 Più Diametro Della Sfera Di Giunzione) -->
-        <origin xyz="0 0 ${l1 + (jointRadius * 2)}" rpy="0 0 0"/>
+        <origin xyz="0 0 ${jointRadius + l1 + jointRadius}" rpy="0 0 0"/>
         <axis xyz="0 1 0"/>
         <!-- DD Movimento Da -90 gradi a +45 gradi Per Evitare Collisioni -->
@@ -124,5 +124,5 @@
         <visual>
             <!-- DD Posizionamento Della Guida Del Prismatico All'Estremità Del Secondo Braccio (Lunghezza L2 Più Diametro Sfera) -->
-            <origin xyz="${l2 + (jointRadius * 2)} 0 0" rpy="0 0 0"/>
+            <origin xyz="${jointRadius + l2 + (boxSize/2)} 0 0" rpy="0 0 0"/>
             <geometry>
                 <box size="${boxSize} ${boxSize} ${boxSize}"/>

Commit message: Fatta Cinematica Inversa In Test.md Da Implementare In inverseKinematics

File: urdf/manipolatoreRRP.urdf.xacro (robot description, xacro)
@@ -29,14 +29,14 @@
 <xacro:macro name="colorDef">
       <material name="baseColor">
-            <color rgba="0.22 0.24 0.26 1.0"/>
+            <color rgba="0.22 0.24 0.26 1"/>
       </material>
       <material name="linkColor">
-            <color rgba="0.65 0.65 0.65 1.0"/>
+            <color rgba="0.65 0.65 0.65 1"/>
       </material>
       <material name="jointColor">
-            <color rgba="0.95 0.72 0.08 1.0"/>
+            <color rgba="0.95 0.72 0.08 0.75"/>
       </material>
       <material name="endEffectorColor">
-            <color rgba="0.8 0.12 0.12 1.0"/>
+            <color rgba="0.8 0.12 0.12 1"/>
       </material>
 </xacro:macro>
@@ -136,6 +136,6 @@
         <parent link="RF1"/>
         <child link="RF2"/>
-        <!-- DD Posizionamento Sull'Asse Della Guida All'Estremità Del Secondo Braccio (Lunghezza L2 Più Diametro Sfera) -->
-        <origin xyz="${l2 + (jointRadius * 2)} 0 0" rpy="0 0 0"/>
+        <!-- DD Posizionamento Sull'Asse Della Guida All'Estremità Del Secondo Braccio (Raggio Sfera + Lunghezza L2 + Metà Dimensione Box) -->
+        <origin xyz="${jointRadius + l2 + (boxSize/2)} 0 0" rpy="0 0 0"/>
         <axis xyz="0 0 1"/>
         <limit effort="100" velocity="1.0" lower="0" upper="${l3 - (eeFingerLength)}"/>

Commit message: Sistemato File XACRO Per Fare In Modo Che I Solidi Si Sovrappongano

File: urdf/manipolatoreRRP.urdf.xacro (robot description, xacro)
@@ -17,5 +17,5 @@
 <!-- BB Giunti -->
 <!-- CC Non E Piu Necessario Definire La Proprieta Perche Gia Presente Di Default In Xacro -->
-<!-- <xacro:property name="pi" value="3.14159265359" /> -->
+<!-- <xacro:property name="pi" value="3.14159erm265359" /> -->
 <xacro:property name="jointRadius" value="${robotParams['jointRadius']}" />     <!-- Raggio Sfere Giunti Revolute (Diametro 10cm) -->
 <xacro:property name="boxSize" value="${robotParams['boxSize']}" />             <!-- Dimensione Box Giunto Prismatico (Lato 11cm) -->
@@ -77,5 +77,5 @@
         <visual>
             <!-- DD Sfera Centrata Sull'Asse Di Rotazione E Sollevata Di Metà Raggio Per Poggiarla Sulla Base -->
-            <origin xyz="0 0 ${jointRadius / 2.0}" rpy="0 0 0"/>
+            <origin xyz="0 0 ${jointRadius}" rpy="0 0 0"/>
             <geometry>
                 <sphere radius="${jointRadius}"/>
@@ -84,6 +84,6 @@
         </visual>
         <visual>
-            <!-- DD Traslazione Di Metà Colonna Più Raggio Sfera Per Evitare Che Entri Dentro La Base -->
-            <origin xyz="0 0 ${(l1 / 2.0) + jointRadius}" rpy="0 0 0"/>
+            <!-- DD Traslazione Di Metà Lunghezza Più Diametro Sfera Per Evitare Che Entri Dentro -->
+            <origin xyz="0 0 ${(l1 / 2.0) + (2 * jointRadius)}" rpy="0 0 0"/>
             <geometry>
                     <cylinder radius="${linkRadius}" length="${l1}" />
@@ -97,6 +97,7 @@
         <parent link="RF0"/>
         <child link="RF1"/>
-        <!-- DD Posizionamento In Cima Al Primo Link (Altezza L1 Più Diametro Della Sfera Di Giunzione) -->
-        <origin xyz="0 0 ${jointRadius + l1 + jointRadius}" rpy="0 0 0"/>
+        <!-- DD Posizionamento In Cima Al Primo Link -->
+        <!-- DD Diametro Sfera Giunto 1 + Lunghezza Link 1 + Raggio Sfera Giunto 2 -->
+        <origin xyz="0 0 ${2*jointRadius + l1 + jointRadius}" rpy="0 0 0"/>
         <axis xyz="0 1 0"/>
         <!-- DD Movimento Da -90 gradi a +45 gradi Per Evitare Collisioni -->
@@ -144,6 +145,7 @@
     <link name="RF2">
         <visual>
-            <!-- DD Asta Centrata Nell'Origine Del Box E Spostata Di Metà Lunghezza E Orientata Verticalmente Per Scorrere Lungo Z -->
-            <origin xyz="0 0 ${-l3/2}" rpy="0 0 0"/>
+            <!-- DD Link Centrato Nell'Origine Del Box Orientato Verticalmente Per Scorrere Lungo Z -->
+            <!-- DD Spostato Di Metà Lunghezza Lato Box + Meta Lunghezza Link -->
+            <origin xyz="0 0 ${-(l3/2 + boxSize/2)}" rpy="0 0 0"/>
             <geometry>
                     <cylinder radius="${linkRadius}" length="${l3}" />
@@ -157,6 +159,7 @@
         <parent link="RF2"/>
         <child link="endEffector"/>
-        <!-- DD Spostato Sulla Punta Inferiore Dell'Asta E Ruotato Di Centottanta Gradi Su Roll -->
-        <origin xyz="0 0 -${l3}" rpy="${pi} 0 0"/>
+        <!-- DD Ruotato Verso Il Basso Di 180° -->
+        <!-- DD Spostato In Basso Di Metà Lunghezza Lato Box + Lunghezza Del Link -->
+        <origin xyz="0 0 ${-(boxSize/2 + l3)}" rpy="${pi} 0 0"/>
         <axis xyz="0 0 1"/>
     </joint>

Commit message: Cinematica Inversa Finita In Appunti_Latex

File: urdf/manipolatoreRRP.urdf.xacro (robot description, xacro)
@@ -140,5 +140,5 @@
         <origin xyz="${jointRadius + l2 + (boxSize/2)} 0 0" rpy="0 0 0"/>
         <axis xyz="0 0 1"/>
-        <limit effort="100" velocity="1.0" lower="0" upper="${l3 - (eeFingerLength)}"/>
+        <limit effort="100" velocity="1.0" lower="0" upper="${l3}"/>
     </joint>
     <!-- BB Cilindro Di Scorrimento (Link 2) -->
@@ -147,5 +147,5 @@
             <!-- DD Link Centrato Nell'Origine Del Box Orientato Verticalmente Per Scorrere Lungo Z -->
             <!-- DD Spostato Di Metà Lunghezza Lato Box + Meta Lunghezza Link -->
-            <origin xyz="0 0 ${-(l3/2 + boxSize/2)}" rpy="0 0 0"/>
+            <origin xyz="0 0 -${(l3/2) + (boxSize/2)}" rpy="0 0 0"/>
             <geometry>
                     <cylinder radius="${linkRadius}" length="${l3}" />
